Commit message: For ROS2
For ROS2

File: TAYO_test_description/urdf/TAYO_test.xacro (robot description, xacro)
@@ -13,5 +13,5 @@
     <origin xyz="0 0 0" rpy="0 0 0"/>
     <geometry>
-      <mesh filename="package://TAYO_test_description/meshes/base_link.stl" scale="0.001 0.001 0.001"/>
+      <mesh filename="file://$(find TAYO_test_description)/meshes/base_link.stl" scale="0.001 0.001 0.001"/>
     </geometry>
     <material name="silver"/>
@@ -20,5 +20,5 @@
     <origin xyz="0 0 0" rpy="0 0 0"/>
     <geometry>
-      <mesh filename="package://TAYO_test_description/meshes/base_link.stl" scale="0.001 0.001 0.001"/>
+      <mesh filename="file://$(find TAYO_test_description)/meshes/base_link.stl" scale="0.001 0.001 0.001"/>
     </geometry>
   </collision>
@@ -33,5 +33,5 @@
     <origin xyz="-0.0 -0.12 -0.065" rpy="0 0 0"/>
     <geometry>
-      <mesh filename="package://TAYO_test_description/meshes/left_wheel_1.stl" scale="0.001 0.001 0.001"/>
+      <mesh filename="file://$(find TAYO_test_description)/meshes/left_wheel_1.stl" scale="0.001 0.001 0.001"/>
     </geometry>
     <material name="silver"/>
@@ -40,5 +40,5 @@
     <origin xyz="-0.0 -0.12 -0.065" rpy="0 0 0"/>
     <geometry>
-      <mesh filename="package://TAYO_test_description/meshes/left_wheel_1.stl" scale="0.001 0.001 0.001"/>
+      <mesh filename="file://$(find TAYO_test_description)/meshes/left_wheel_1.stl" scale="0.001 0.001 0.001"/>
     </geometry>
   </collision>
@@ -53,5 +53,5 @@
     <origin xyz="-0.0 0.12 -0.065" rpy="0 0 0"/>
     <geometry>
-      <mesh filename="package://TAYO_test_description/meshes/right_wheel_1.stl" scale="0.001 0.001 0.001"/>
+      <mesh filename="file://$(find TAYO_test_description)/meshes/right_wheel_1.stl" scale="0.001 0.001 0.001"/>
     </geometry>
     <material name="silver"/>
@@ -60,5 +60,5 @@
     <origin xyz="-0.0 0.12 -0.065" rpy="0 0 0"/>
     <geometry>
-      <mesh filename="package://TAYO_test_description/meshes/right_wheel_1.stl" scale="0.001 0.001 0.001"/>
+      <mesh filename="file://$(find TAYO_test_description)/meshes/right_wheel_1.stl" scale="0.001 0.001 0.001"/>
     </geometry>
   </collision>
@@ -73,5 +73,5 @@
     <origin xyz="-0.0 -0.0 -0.1697" rpy="0 0 0"/>
     <geometry>
-      <mesh filename="package://TAYO_test_description/meshes/lidar_1.stl" scale="0.001 0.001 0.001"/>
+      <mesh filename="file://$(find TAYO_test_description)/meshes/lidar_1.stl" scale="0.001 0.001 0.001"/>
     </geometry>
     <material name="silver"/>
@@ -80,5 +80,5 @@
     <origin xyz="-0.0 -0.0 -0.1697" rpy="0 0 0"/>
     <geometry>
-      <mesh filename="package://TAYO_test_description/meshes/lidar_1.stl" scale="0.001 0.001 0.001"/>
+      <mesh filename="file://$(find TAYO_test_description)/meshes/lidar_1.stl" scale="0.001 0.001 0.001"/>
     </geometry>
   </collision>
@@ -93,5 +93,5 @@
     <origin xyz="-0.0 -0.0 -0.217" rpy="0 0 0"/>
     <geometry>
-      <mesh filename="package://TAYO_test_description/meshes/imu_1.stl" scale="0.001 0.001 0.001"/>
+      <mesh filename="file://$(find TAYO_test_description)/meshes/imu_1.stl" scale="0.001 0.001 0.001"/>
     </geometry>
     <material name="silver"/>
@@ -100,5 +100,5 @@
     <origin xyz="-0.0 -0.0 -0.217" rpy="0 0 0"/>
     <geometry>
-      <mesh filename="package://TAYO_test_description/meshes/imu_1.stl" scale="0.001 0.001 0.001"/>
+      <mesh filename="file://$(find TAYO_test_description)/meshes/imu_1.stl" scale="0.001 0.001 0.001"/>
     </geometry>
   </collision>
@@ -113,5 +113,5 @@
     <origin xyz="-0.094 -0.0 -1.12" rpy="0 0 0"/>
     <geometry>
-      <mesh filename="package://TAYO_test_description/meshes/camera_1.stl" scale="0.001 0.001 0.001"/>
+      <mesh filename="file://$(find TAYO_test_description)/meshes/camera_1.stl" scale="0.001 0.001 0.001"/>
     </geometry>
     <material name="silver"/>
@@ -120,5 +120,5 @@
     <origin xyz="-0.094 -0.0 -1.12" rpy="0 0 0"/>
     <geometry>
-      <mesh filename="package://TAYO_test_description/meshes/camera_1.stl" scale="0.001 0.001 0.001"/>
+      <mesh filename="file://$(find TAYO_test_description)/meshes/camera_1.stl" scale="0.001 0.001 0.001"/>
     </geometry>
   </collision>
@@ -133,5 +133,5 @@
     <origin xyz="-0.1 -0.0 -0.593" rpy="0 0 0"/>
     <geometry>
-      <mesh filename="package://TAYO_test_description/meshes/actuator_1.stl" scale="0.001 0.001 0.001"/>
+      <mesh filename="file://$(find TAYO_test_description)/meshes/actuator_1.stl" scale="0.001 0.001 0.001"/>
     </geometry>
     <material name="silver"/>
@@ -140,9 +140,9 @@
     <origin xyz="-0.1 -0.0 -0.593" rpy="0 0 0"/>
     <geometry>
-      <mesh filename="package://TAYO_test_description/meshes/actuator_1.stl" scale="0.001 0.001 0.001"/>
+      <mesh filename="file://$(find TAYO_test_description)/meshes/actuator_1.stl" scale="0.001 0.001 0.001"/>
     </geometry>
   </collision>
 </link>
-<joint name="ȸ�� 1" type="continuous">
+<joint name="Revolute 1" type="continuous">
   <origin xyz="0.0 0.12 0.065" rpy="0 0 0"/>
   <parent link="base_link"/>
@@ -150,5 +150,5 @@
   <axis xyz="0.0 1.0 0.0"/>
 </joint>
-<joint name="ȸ�� 2" type="continuous">
+<joint name="Revolute 2" type="continuous">
   <origin xyz="0.0 -0.12 0.065" rpy="0 0 0"/>
   <parent link="base_link"/>
@@ -156,20 +156,20 @@
   <axis xyz="0.0 -1.0 0.0"/>
 </joint>
-<joint name="��ü 3" type="fixed">
+<joint name="Rigid 3" type="fixed">
   <origin xyz="0.0 0.0 0.1697" rpy="0 0 0"/>
   <parent link="base_link"/>
   <child link="lidar_1"/>
 </joint>
-<joint name="��ü 4" type="fixed">
+<joint name="Rigid 4" type="fixed">
   <origin xyz="0.0 0.0 0.217" rpy="0 0 0"/>
   <parent link="base_link"/>
   <child link="imu_1"/>
 </joint>
-<joint name="��ü 5" type="fixed">
+<joint name="Rigid 5" type="fixed">
   <origin xyz="-0.006 0.0 0.527" rpy="0 0 0"/>
   <parent link="actuator_1"/>
   <child link="camera_1"/>
 </joint>
-<joint name="�����̴� 6" type="prismatic">
+<joint name="Slider 6" type="prismatic">
   <origin xyz="0.1 0.0 0.593" rpy="0 0 0"/>
   <parent link="base_link"/>

Commit message: Edit materials.xacro
Add colors

File: TAYO_test_description/urdf/TAYO_test.xacro (robot description, xacro)
@@ -24,4 +24,24 @@
   </collision>
 </link>
+<link name="right_wheel_1">
+  <inertial>
+    <origin xyz="-2.14128073229365e-17 -0.03200000000000003 0.0" rpy="0 0 0"/>
+    <mass value="0.7900225877835323"/>
+    <inertia ixx="0.001104" iyy="0.001669" izz="0.001104" ixy="-0.0" iyz="-0.0" ixz="-0.0"/>
+  </inertial>
+  <visual>
+    <origin xyz="-0.0 0.12 -0.065" rpy="0 0 0"/>
+    <geometry>
+      <mesh filename="file://$(find TAYO_test_description)/meshes/right_wheel_1.stl" scale="0.001 0.001 0.001"/>
+    </geometry>
+    <material name="black"/>
+  </visual>
+  <collision>
+    <origin xyz="-0.0 0.12 -0.065" rpy="0 0 0"/>
+    <geometry>
+      <mesh filename="file://$(find TAYO_test_description)/meshes/right_wheel_1.stl" scale="0.001 0.001 0.001"/>
+    </geometry>
+  </collision>
+</link>
 <link name="left_wheel_1">
   <inertial>
@@ -35,5 +55,5 @@
       <mesh filename="file://$(find TAYO_test_description)/meshes/left_wheel_1.stl" scale="0.001 0.001 0.001"/>
     </geometry>
-    <material name="silver"/>
+    <material name="black"/>
   </visual>
   <collision>
@@ -44,21 +64,21 @@
   </collision>
 </link>
-<link name="right_wheel_1">
+<link name="actuator_1">
   <inertial>
-    <origin xyz="-2.14128073229365e-17 -0.03200000000000003 0.0" rpy="0 0 0"/>
-    <mass value="0.7900225877835323"/>
-    <inertia ixx="0.001104" iyy="0.001669" izz="0.001104" ixy="-0.0" iyz="-0.0" ixz="-0.0"/>
+    <origin xyz="0.028488110282179235 -1.0854817842170162e-16 0.28699337976007466" rpy="0 0 0"/>
+    <mass value="14.478426699691301"/>
+    <inertia ixx="0.629374" iyy="0.316333" izz="0.325608" ixy="-0.0" iyz="-0.0" ixz="0.004938"/>
   </inertial>
   <visual>
-    <origin xyz="-0.0 0.12 -0.065" rpy="0 0 0"/>
+    <origin xyz="-0.1 -0.0 -0.818" rpy="0 0 0"/>
     <geometry>
-      <mesh filename="file://$(find TAYO_test_description)/meshes/right_wheel_1.stl" scale="0.001 0.001 0.001"/>
+      <mesh filename="file://$(find TAYO_test_description)/meshes/actuator_1.stl" scale="0.001 0.001 0.001"/>
     </geometry>
-    <material name="silver"/>
+    <material name="orange"/>
   </visual>
   <collision>
-    <origin xyz="-0.0 0.12 -0.065" rpy="0 0 0"/>
+    <origin xyz="-0.1 -0.0 -0.818" rpy="0 0 0"/>
     <geometry>
-      <mesh filename="file://$(find TAYO_test_description)/meshes/right_wheel_1.stl" scale="0.001 0.001 0.001"/>
+      <mesh filename="file://$(find TAYO_test_description)/meshes/actuator_1.stl" scale="0.001 0.001 0.001"/>
     </geometry>
   </collision>
@@ -75,5 +95,5 @@
       <mesh filename="file://$(find TAYO_test_description)/meshes/lidar_1.stl" scale="0.001 0.001 0.001"/>
     </geometry>
-    <material name="silver"/>
+    <material name="red"/>
   </visual>
   <collision>
@@ -95,5 +115,5 @@
       <mesh filename="file://$(find TAYO_test_description)/meshes/imu_1.stl" scale="0.001 0.001 0.001"/>
     </geometry>
-    <material name="silver"/>
+    <material name="blue"/>
   </visual>
   <collision>
@@ -106,17 +126,17 @@
 <link name="camera_1">
   <inertial>
-    <origin xyz="0.012499999999999983 1.608339750033895e-17 0.0" rpy="0 0 0"/>
+    <origin xyz="0.012499999999999983 2.052428959883958e-17 0.0" rpy="0 0 0"/>
     <mass value="0.13872095061007444"/>
-    <inertia ixx="1.6e-05" iyy="1.5e-05" izz="1.5e-05" ixy="0.0" iyz="0.0" ixz="0.0"/>
+    <inertia ixx="1.6e-05" iyy="1.5e-05" izz="1.5e-05" ixy="0.0" iyz="0.0" ixz="-0.0"/>
   </inertial>
   <visual>
-    <origin xyz="-0.094 -0.0 -1.12" rpy="0 0 0"/>
+    <origin xyz="-0.094 -0.0 -1.32" rpy="0 0 0"/>
     <geometry>
       <mesh filename="file://$(find TAYO_test_description)/meshes/camera_1.stl" scale="0.001 0.001 0.001"/>
     </geometry>
-    <material name="silver"/>
+    <material name="red"/>
   </visual>
   <collision>
-    <origin xyz="-0.094 -0.0 -1.12" rpy="0 0 0"/>
+    <origin xyz="-0.094 -0.0 -1.32" rpy="0 0 0"/>
     <geometry>
       <mesh filename="file://$(find TAYO_test_description)/meshes/camera_1.stl" scale="0.001 0.001 0.001"/>
@@ -124,25 +144,11 @@
   </collision>
 </link>
-<link name="actuator_1">
-  <inertial>
-    <origin xyz="0.028488110282179235 -1.0854817842170162e-16 0.31199337976007446" rpy="0 0 0"/>
-    <mass value="14.478426699691301"/>
-    <inertia ixx="0.629374" iyy="0.316333" izz="0.325608" ixy="-0.0" iyz="-0.0" ixz="0.004938"/>
-  </inertial>
-  <visual>
-    <origin xyz="-0.1 -0.0 -0.593" rpy="0 0 0"/>
-    <geometry>
-      <mesh filename="file://$(find TAYO_test_description)/meshes/actuator_1.stl" scale="0.001 0.001 0.001"/>
-    </geometry>
-    <material name="silver"/>
-  </visual>
-  <collision>
-    <origin xyz="-0.1 -0.0 -0.593" rpy="0 0 0"/>
-    <geometry>
-      <mesh filename="file://$(find TAYO_test_description)/meshes/actuator_1.stl" scale="0.001 0.001 0.001"/>
-    </geometry>
-  </collision>
-</link>
-<joint name="Revolute 1" type="continuous">
+<joint name="Revolute 7" type="continuous">
+  <origin xyz="0.0 -0.12 0.065" rpy="0 0 0"/>
+  <parent link="base_link"/>
+  <child link="right_wheel_1"/>
+  <axis xyz="0.0 -1.0 0.0"/>
+</joint>
+<joint name="Revolute 8" type="continuous">
   <origin xyz="0.0 0.12 0.065" rpy="0 0 0"/>
   <parent link="base_link"/>
@@ -150,31 +156,25 @@
   <axis xyz="0.0 1.0 0.0"/>
 </joint>
-<joint name="Revolute 2" type="continuous">
-  <origin xyz="0.0 -0.12 0.065" rpy="0 0 0"/>
+<joint name="Slider 9" type="prismatic">
+  <origin xyz="0.1 0.0 0.818" rpy="0 0 0"/>
   <parent link="base_link"/>
-  <child link="right_wheel_1"/>
-  <axis xyz="0.0 -1.0 0.0"/>
+  <child link="actuator_1"/>
+  <axis xyz="0.0 0.0 -1.0"/>
+  <limit upper="0.2" lower="-0.2" effort="100" velocity="100"/>
 </joint>
-<joint name="Rigid 3" type="fixed">
+<joint name="Rigid 10" type="fixed">
   <origin xyz="0.0 0.0 0.1697" rpy="0 0 0"/>
   <parent link="base_link"/>
   <child link="lidar_1"/>
 </joint>
-<joint name="Rigid 4" type="fixed">
+<joint name="Rigid 11" type="fixed">
   <origin xyz="0.0 0.0 0.217" rpy="0 0 0"/>
   <parent link="base_link"/>
   <child link="imu_1"/>
 </joint>
-<joint name="Rigid 5" type="fixed">
-  <origin xyz="-0.006 0.0 0.527" rpy="0 0 0"/>
+<joint name="Rigid 12" type="fixed">
+  <origin xyz="-0.006 0.0 0.502" rpy="0 0 0"/>
   <parent link="actuator_1"/>
   <child link="camera_1"/>
 </joint>
-<joint name="Slider 6" type="prismatic">
-  <origin xyz="0.1 0.0 0.593" rpy="0 0 0"/>
-  <parent link="base_link"/>
-  <child link="actuator_1"/>
-  <axis xyz="0.0 0.0 1.0"/>
-  <limit upper="0.0" lower="0.0" effort="100" velocity="100"/>
-</joint>
 </robot>

File: TAYO_test_description/urdf/materials.xacro (robot description, xacro)
@@ -4,3 +4,15 @@
   <color rgba="0.700 0.700 0.700 1.000"/>
 </material>
+<material name="black">
+  <color rgba="0.000 0.000 0.000 1.000"/>
+</material>
+<material name="blue">
+  <color rgba="0.000 0.000 0.800 1.000"/>
+</material>
+<material name="orange">
+  <color rgba="1.000 0.4235 0.0392 1.000"/>
+</material>
+<material name="red">
+  <color rgba="0.800 0.000 0.000 1.000"/>
+</material>
 </robot>
